Commit message: Update robot.urdf.xacro

File: robot_description/urdf/robot.urdf.xacro (robot description, xacro)
@@ -33,4 +33,7 @@
   <xacro:property name="wheel_mass" value="0.5"/>
   <xacro:property name="wheel_y_offset" value="0.23"/>
+  <!-- caster wheel -->
+  <xacro:property name="caster_radius" value="0.05"/>
+  <xacro:property name="caster_mass" value="0.1"/>
   <link name="base_footprint"/>
   <joint name="base_footprint_joint" type="fixed">
@@ -225,3 +228,25 @@
   <xacro:wheel prefix="left"  y_reflect="1"/>
   <xacro:wheel prefix="right" y_reflect="-1"/>
+<joint name="caster_wheel_joint" type="fixed">
+  <parent link="base_link"/>
+  <child link="caster_wheel_link"/>
+  <!-- rear of the chassis, centered in y, dropped so the sphere still touches the ground -->
+  <origin xyz="${-step1_length/2 + caster_radius} 0 ${-(wheel_radius - caster_radius)}" rpy="0 0 0"/>
+</joint>
+<link name="caster_wheel_link">
+  <visual>
+    <geometry><sphere radius="${caster_radius}"/></geometry>
+    <material name="caster_red"><color rgba="1.0 0.0 0.0 1.0"/></material>
+  </visual>
+  <collision>
+    <geometry><sphere radius="${caster_radius}"/></geometry>
+  </collision>
+  <inertial>
+    <mass value="${caster_mass}"/>
+    <origin xyz="0 0 0" rpy="0 0 0"/>
+    <inertia ixx="${(2/5)*caster_mass*caster_radius*caster_radius}" ixy="0.0" ixz="0.0"
+             iyy="${(2/5)*caster_mass*caster_radius*caster_radius}" iyz="0.0"
+             izz="${(2/5)*caster_mass*caster_radius*caster_radius}"/>
+  </inertial>
+</link>
 </robot>

Commit message: Update robot.urdf.xacro

File: robot_description/urdf/robot.urdf.xacro (robot description, xacro)
@@ -5,7 +5,7 @@
   <!-- ============================================================ -->
   <!-- PYRAMID CHASSIS - 3 stacked steps, Egyptian flag color order  -->
-  <!-- (red bottom, white middle, black top - widest to narrowest)   -->
-  <!-- ============================================================ -->
-  <!-- Step 1 - base / bottom step (RED) -->
+  <!-- (Black bottom, white middle, Red top - widest to narrowest)   -->
+  <!-- ============================================================ -->
+  <!-- Step 1 - base / bottom step (Black) -->
   <xacro:property name="step1_length" value="0.6"/>
   <xacro:property name="step1_width" value="0.4"/>
@@ -17,5 +17,5 @@
   <xacro:property name="step2_height" value="0.12"/>
   <xacro:property name="step2_mass" value="1.5"/>
-  <!-- Step 3 - top step (BLACK) -->
+  <!-- Step 3 - top step (Red) -->
   <xacro:property name="step3_length" value="0.26"/>
   <xacro:property name="step3_width" value="0.18"/>
@@ -42,27 +42,36 @@
     <origin xyz="0 0 ${wheel_radius}" rpy="0 0 0"/>
   </joint>
-  <!-- ============== STEP 1 (base_link) - RED ============== -->
-  <link name="base_link">
-    <visual>
-      <geometry>
-        <box size="${step1_length} ${step1_width} ${step1_height}"/>
-      </geometry>
-      <material name="step1_red">
-        <color rgba="${color_black}"/>
-      </material>
-    </visual>
-    <collision>
-      <geometry>
-        <box size="${step1_length} ${step1_width} ${step1_height}"/>
-      </geometry>
-    </collision>
-    <inertial>
-      <mass value="${step1_mass}"/>
-      <origin xyz="0 0 0" rpy="0 0 0"/>
-      <inertia ixx="${(1/12) * step1_mass * (step1_width*step1_width + step1_height*step1_height)}" ixy="0.0" ixz="0.0"
-               iyy="${(1/12) * step1_mass * (step1_length*step1_length + step1_height*step1_height)}" iyz="0.0"
-               izz="${(1/12) * step1_mass * (step1_length*step1_length + step1_width*step1_width)}"/>
-    </inertial>
-  </link>
+  <!-- ============================================================ -->
+  <!-- CHASSIS STEP MACRO - box link (visual/collision/inertial)     -->
+  <!-- identical structure for all 3 steps, only size/mass/color     -->
+  <!-- differ, so it's parameterized the same way the wheel is.      -->
+  <!-- ============================================================ -->
+    <xacro:macro name="chassis_step" params="name length width height mass color">
+    <link name="${name}">
+      <visual>
+        <geometry>
+          <box size="${length} ${width} ${height}"/>
+        </geometry>
+        <material name="${name}_material">
+          <color rgba="${color}"/>
+        </material>
+      </visual>
+      <collision>
+        <geometry>
+          <box size="${length} ${width} ${height}"/>
+        </geometry>
+      </collision>
+      <inertial>
+        <mass value="${mass}"/>
+        <origin xyz="0 0 0" rpy="0 0 0"/>
+        <inertia ixx="${(1/12) * mass * (width*width + height*height)}" ixy="0.0" ixz="0.0"
+                 iyy="${(1/12) * mass * (length*length + height*height)}" iyz="0.0"
+                 izz="${(1/12) * mass * (length*length + width*width)}"/>
+      </inertial>
+    </link>
+  </xacro:macro>
+  <!-- ============== STEP 1 (base_link) - Black ============== -->
+  <xacro:chassis_step name="base_link" length="${step1_length}" width="${step1_width}"
+                       height="${step1_height}" mass="${step1_mass}" color="${color_black}"/>
   <!-- ============== STEP 2 (middle_step_link) - WHITE ============== -->
   <joint name="middle_step_joint" type="fixed">
@@ -71,27 +80,7 @@
     <origin xyz="0 0 ${step1_height/2 + step2_height/2}" rpy="0 0 0"/>
   </joint>
-  <link name="middle_step_link">
-    <visual>
-      <geometry>
-        <box size="${step2_length} ${step2_width} ${step2_height}"/>
-      </geometry>
-      <material name="step2_white">
-        <color rgba="${color_white}"/>
-      </material>
-    </visual>
-    <collision>
-      <geometry>
-        <box size="${step2_length} ${step2_width} ${step2_height}"/>
-      </geometry>
-    </collision>
-    <inertial>
-      <mass value="${step2_mass}"/>
-      <origin xyz="0 0 0" rpy="0 0 0"/>
-      <inertia ixx="${(1/12) * step2_mass * (step2_width*step2_width + step2_height*step2_height)}" ixy="0.0" ixz="0.0"
-               iyy="${(1/12) * step2_mass * (step2_length*step2_length + step2_height*step2_height)}" iyz="0.0"
-               izz="${(1/12) * step2_mass * (step2_length*step2_length + step2_width*step2_width)}"/>
-    </inertial>
-  </link>
-  <!-- ============== STEP 3 (top_step_link) - BLACK ============== -->
+  <xacro:chassis_step name="middle_step_link" length="${step2_length}" width="${step2_width}"
+                       height="${step2_height}" mass="${step2_mass}" color="${color_white}"/>
+  <!-- ============== STEP 3 (top_step_link) - RED ============== -->
   <joint name="top_step_joint" type="fixed">
     <parent link="middle_step_link"/>
@@ -99,26 +88,6 @@
     <origin xyz="0 0 ${step2_height/2 + step3_height/2}" rpy="0 0 0"/>
   </joint>
-  <link name="top_step_link">
-    <visual>
-      <geometry>
-        <box size="${step3_length} ${step3_width} ${step3_height}"/>
-      </geometry>
-      <material name="step3_black">
-        <color rgba="${color_red}"/>
-      </material>
-    </visual>
-    <collision>
-      <geometry>
-        <box size="${step3_length} ${step3_width} ${step3_height}"/>
-      </geometry>
-    </collision>
-    <inertial>
-      <mass value="${step3_mass}"/>
-      <origin xyz="0 0 0" rpy="0 0 0"/>
-      <inertia ixx="${(1/12) * step3_mass * (step3_width*step3_width + step3_height*step3_height)}" ixy="0.0" ixz="0.0"
-               iyy="${(1/12) * step3_mass * (step3_length*step3_length + step3_height*step3_height)}" iyz="0.0"
-               izz="${(1/12) * step3_mass * (step3_length*step3_length + step3_width*step3_width)}"/>
-    </inertial>
-  </link>
+  <xacro:chassis_step name="top_step_link" length="${step3_length}" width="${step3_width}"
+                       height="${step3_height}" mass="${step3_mass}" color="${color_red}"/>
   <!-- ============================================================ -->
   <!-- CAMERA - mounted on the MIDDLE (white) step, colored GOLD     -->

Commit message: Update robot.urdf.xacro

File: robot_description/urdf/robot.urdf.xacro (robot description, xacro)
@@ -8,18 +8,18 @@
   <!-- ============================================================ -->
   <!-- Step 1 - base / bottom step (Black) -->
-  <xacro:property name="step1_length" value="0.6"/>
-  <xacro:property name="step1_width" value="0.4"/>
-  <xacro:property name="step1_height" value="0.15"/>
-  <xacro:property name="step1_mass" value="3.0"/>
+  <xacro:property name="step1_length" value="0.2"/>
+  <xacro:property name="step1_width" value="0.15"/>
+  <xacro:property name="step1_height" value="0.05"/>
+  <xacro:property name="step1_mass" value="0.3"/>
   <!-- Step 2 - middle step (WHITE) -->
-  <xacro:property name="step2_length" value="0.42"/>
-  <xacro:property name="step2_width" value="0.28"/>
-  <xacro:property name="step2_height" value="0.12"/>
-  <xacro:property name="step2_mass" value="1.5"/>
+  <xacro:property name="step2_length" value="0.15"/>
+  <xacro:property name="step2_width" value="0.1"/>
+  <xacro:property name="step2_height" value="0.05"/>
+  <xacro:property name="step2_mass" value="0.15"/>
   <!-- Step 3 - top step (Red) -->
-  <xacro:property name="step3_length" value="0.26"/>
-  <xacro:property name="step3_width" value="0.18"/>
-  <xacro:property name="step3_height" value="0.10"/>
-  <xacro:property name="step3_mass" value="0.8"/>
+  <xacro:property name="step3_length" value="0.1"/>
+  <xacro:property name="step3_width" value="0.05"/>
+  <xacro:property name="step3_height" value="0.03"/>
+  <xacro:property name="step3_mass" value="0.08"/>
   <!-- Colors -->
   <xacro:property name="color_red" value="0.80 0.07 0.15 1.0"/>     <!-- Egyptian flag red -->
@@ -29,10 +29,10 @@
   <xacro:property name="color_wheel" value="0.55 0.35 0.12 1.0"/>    <!-- antique bronze, complements the gold -->
   <!-- Wheels -->
-  <xacro:property name="wheel_radius" value="0.1"/>
-  <xacro:property name="wheel_width" value="0.05"/>
-  <xacro:property name="wheel_mass" value="0.5"/>
-  <xacro:property name="wheel_y_offset" value="0.23"/>
+  <xacro:property name="wheel_radius" value="0.0325"/>
+  <xacro:property name="wheel_width" value="0.026"/>
+  <xacro:property name="wheel_mass" value="0.1"/>
+  <xacro:property name="wheel_y_offset" value="0.088"/>
   <!-- caster wheel -->
-  <xacro:property name="caster_radius" value="0.05"/>
+  <xacro:property name="caster_radius" value="0.015"/>
   <xacro:property name="caster_mass" value="0.1"/>
   <link name="base_footprint"/>
@@ -158,5 +158,5 @@
     <parent link="top_step_link"/>
     <child link="lidar_link"/>
-    <origin xyz="0 0 ${step3_height/2 + 0.02}" rpy="0 0 0"/>
+    <origin xyz="0.02 0 ${step3_height/2 + 0.03}" rpy="0 0 0"/>
   </joint>
   <!-- ============================================================ -->
@@ -167,5 +167,5 @@
       <parent link="base_link"/>
       <child link="${prefix}_wheel_link"/>
-      <origin xyz="0 ${y_reflect * wheel_y_offset} 0" rpy="0 0 0"/>
+      <origin xyz="${-step1_length/2+2*wheel_radius} ${y_reflect * wheel_y_offset} 0" rpy="0 0 0"/>
       <axis xyz="0 1 0"/>
     </joint>
@@ -201,5 +201,5 @@
   <child link="caster_wheel_link"/>
   <!-- rear of the chassis, centered in y, dropped so the sphere still touches the ground -->
-  <origin xyz="${-step1_length/2 + caster_radius} 0 ${-(wheel_radius - caster_radius)}" rpy="0 0 0"/>
+  <origin xyz="${step1_length/2 - 2*caster_radius} 0 ${-(wheel_radius - caster_radius)}" rpy="0 0 0"/>
 </joint>
 <link name="caster_wheel_link">
